Commit message: PR2 Dynamic env commit

File: pr2_common/pr2_description/robots/pr2.urdf.xacro (robot description, xacro)
@@ -137,4 +137,5 @@
       <xacro:kinect_prosilica_camera_swept_back_v0 name="head_mount" parent="head_plate_frame" >
         <origin xyz="-0.137376 0 0.091746" rpy="0 0 0" />
+        <!-- <origin xyz="-0.137376 0 0.12" rpy="0 0 0" /> -->
         <!--
               Was -0.1 0 0.09225, -0.138 0 0.09225 looks good front back and sheet metal on bolt pattern,

File: pr2_common/pr2_description/urdf/forearm_v0/forearm.urdf.xacro (robot description, xacro)
@@ -115,4 +115,10 @@
       </collision>
     </link>
+    <joint name="${side}_tip_joint" type="fixed">
+      <origin xyz="0.18 0 0" rpy="0 0 0" />
+      <parent link="${side}_wrist_roll_link"/>
+      <child link="${side}_tip_link"/>
+    </joint>
+    <link name="${side}_tip_link"/>
     <!-- extensions-->
     <xacro:pr2_forearm_gazebo_v0 side="${side}" />

File: pr2_common/pr2_description/urdf/forearm_v0/forearm_moveit.urdf.xacro (robot description, xacro)
@@ -115,4 +115,10 @@
       </collision>
     </link>
+    <!-- <joint name="${side}_tip_joint" type="fixed">
+      <origin xyz="0.18 0 0" rpy="0 0 0" />
+      <parent link="${side}_wrist_roll_link"/>
+      <child link="${side}_tip_link"/>
+    </joint>
+    <link name="${side}_tip_link"/> -->
     <!-- extensions-->
     <xacro:pr2_forearm_gazebo_v0 side="${side}" />
